File: KICAD/Model-U-GCC-V2.kicad_sch (KiCad schematic)
At the start: 5 parts

Commit message: 00000
Parts:
- gave numbers to parts that had none: 5
Changed lines of the file:
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@@
   (symbol (lib_id "Model-U-GCC-V2-rescue:USB_C_Receptacle-Model_S-Model-U-GCC-rescue") (at 95.25 86.36 0) (unit 1)
     (in_bom yes) (on_board yes)
-    (property "Reference" "" (id 0) (at 86.36 59.69 0))
+    (property "Reference" "J1" (id 0) (at 86.36 59.69 0))
     (property "Value" "USB_C_Receptacle" (id 1) (at 95.25 57.15 0))
     (property "Footprint" "Model_S:Shou Han Type-C 24P QCHT" (id 2) (at 99.06 86.36 0)
@@
   (symbol (lib_id "Model-U-GCC-V2-rescue:GND-Model_S-Model-U-GCC-rescue") (at 95.25 129.54 0) (unit 1)
     (in_bom yes) (on_board yes)
-    (property "Reference" "" (id 0) (at 95.25 135.89 0)
+    (property "Reference" "#PWR0122" (id 0) (at 95.25 135.89 0)
       (effects (font (size 1.27 1.27)) hide)
     )
@@
   (symbol (lib_id "Connector_Generic:Conn_01x02") (at 154.94 100.33 0) (mirror y) (unit 1)
     (in_bom yes) (on_board yes)
-    (property "Reference" "" (id 0) (at 152.4 99.06 0))
+    (property "Reference" "J3" (id 0) (at 152.4 99.06 0))
     (property "Value" "Conn_01x02" (id 1) (at 154.94 95.25 0))
     (property "Footprint" "Connector_PinHeader_2.00mm:PinHeader_1x02_P2.00mm_Vertical" (id 2) (at 154.94 100.33 0)
@@
   (symbol (lib_id "Model-U-GCC-V2-rescue:GND-Model_S-Model-U-GCC-rescue") (at 168.91 71.12 270) (unit 1)
     (in_bom yes) (on_board yes)
-    (property "Reference" "" (id 0) (at 162.56 71.12 0)
+    (property "Reference" "#PWR0101" (id 0) (at 162.56 71.12 0)
       (effects (font (size 1.27 1.27)) hide)
     )
@@
   (symbol (lib_id "Device:R") (at 128.27 66.04 270) (unit 1)
     (in_bom yes) (on_board yes)
-    (property "Reference" "" (id 0) (at 128.27 63.5 90))
+    (property "Reference" "R1" (id 0) (at 128.27 63.5 90))
     (property "Value" "5.1k" (id 1) (at 128.27 66.04 90))
     (property "Footprint" "Resistor_SMD:R_0603_1608Metric" (id 2) (at 128.27 64.262 90)
@@
   (symbol (lib_id "Device:R") (at 128.27 68.58 90) (unit 1)
     (in_bom yes) (on_board yes)
-    (property "Reference" "" (id 0) (at 128.27 71.12 90))
+    (property "Reference" "R2" (id 0) (at 128.27 71.12 90))
     (property "Value" "5.1k" (id 1) (at 128.27 68.58 90))
     (property "Footprint" "Resistor_SMD:R_0603_1608Metric" (id 2) (at 128.27 70.358 90)
@@
   (symbol (lib_id "Model-U-GCC-V2-rescue:GND-Model_S-Model-U-GCC-rescue") (at 134.62 71.12 0) (unit 1)
     (in_bom yes) (on_board yes)
-    (property "Reference" "" (id 0) (at 134.62 77.47 0)
+    (property "Reference" "#PWR0103" (id 0) (at 134.62 77.47 0)
       (effects (font (size 1.27 1.27)) hide)
     )
@@
   (symbol (lib_id "Connector_Generic:Conn_01x06") (at 173.99 68.58 0) (unit 1)
     (in_bom yes) (on_board yes)
-    (property "Reference" "" (id 0) (at 176.022 68.7832 0)
+    (property "Reference" "J2" (id 0) (at 176.022 68.7832 0)
       (effects (font (size 1.27 1.27)) (justify left))
     )
@@
   (symbol (lib_id "Model-U-GCC-V2-rescue:GND-Model_S-Model-U-GCC-rescue") (at 168.91 73.66 270) (unit 1)
     (in_bom yes) (on_board yes)
-    (property "Reference" "" (id 0) (at 162.56 73.66 0)
+    (property "Reference" "#PWR0104" (id 0) (at 162.56 73.66 0)
       (effects (font (size 1.27 1.27)) hide)
     )
@@
   (symbol (lib_id "Model-U-GCC-V2-rescue:GND-Model_S-Model-U-GCC-rescue") (at 168.91 76.2 270) (unit 1)
     (in_bom yes) (on_board yes)
-    (property "Reference" "" (id 0) (at 162.56 76.2 0)
+    (property "Reference" "#PWR0105" (id 0) (at 162.56 76.2 0)
       (effects (font (size 1.27 1.27)) hide)
     )
